Commit message: Testing shape transforming

File: data/urdf/shadow_hand_john/sr_description/model_arm_and_hand3.urdf (robot description, URDF)
Before this commit: robot arm_and_hand, 33 links, 32 joints
Links:
- added link shadowarm_base, mass 0.4; collision mesh filename=package://sr_description/arm/model/arm_base.dae scale=0.001 0.001 0.001; visual mesh filename=package://sr_description/arm/model/arm_base.dae scale=0.001 0.001 0.001
- added link shadowarm_trunk, mass 0.5; collision mesh filename=package://sr_description/arm/model/arm_trunk.dae scale=0.001 0.001 0.001; visual mesh filename=package://sr_description/arm/model/arm_trunk.dae scale=0.001 0.001 0.001
- added link shadowarm_upperarm, mass 0.5; collision mesh filename=package://sr_description/arm/model/upper_arm.dae scale=0.001 0.001 0.001; visual mesh filename=package://sr_description/arm/model/upper_arm.dae scale=0.001 0.001 0.001
Joints:
- added joint ShoulderJRotate: type revolute, parent shadowarm_base, child shadowarm_trunk, origin xyz=0 0 0.01 rpy=0.0 0.0 0.0, axis 0 0 1, limit lower=-0.785398163397 upper=1.57079632679 effort=1000.0 velocity=10.0
- added joint ShoulderJSwing: type revolute, parent shadowarm_trunk, child shadowarm_upperarm, origin xyz=0 -0.134 0.5305 rpy=0 -3.14159265359 0.0, axis 0 -1 0, limit lower=0 upper=1.57079632679 effort=1000.0 velocity=10.0
- added joint arm_to_world_fixed: type fixed, parent world, child shadowarm_base, origin xyz=0 -1 1.0 rpy=0 0 0
- joint ElbowJSwing: parent world -> shadowarm_upperarm

File: data/urdf/shadow_hand_john/sr_description/model_forearm_and_hand_JS.urdf (robot description, URDF)
Before this commit: robot arm_and_hand, 33 links, 32 joints
Links:
- removed link shadowarm_lowerarm
Joints:
- joint ElbowJSwing: axis 0 -1 0 -> (none); child shadowarm_lowerarm -> shadowarm_handsupport; limit lower=0.52 upper=2.09439510239 effort=1000.0 velocity=10.0 -> (none); type revolute -> fixed
- joint arm_link: origin xyz=0 0 0 rpy=0 0 2.35619449 -> xyz=0.08 0 0.121 rpy=0 0 2.35619449
