Commit message: Rigid shadow hand modeling done

File: data/urdf/shadow_hand_john/model_arm_and_hand.urdf (robot description, URDF)
Before this commit: robot arm_and_hand, 36 links, 35 joints
Links:
- link ffdistal: geometry collision mesh filename=sr_description/hand/model/F1.dae scale=0.001 0.001 0.001; visual mesh filename=sr_description/hand/model/F1.dae scale=0.001 0.001 0.001
- link ffknuckle: geometry collision box size=0.005 0.005 0.005; visual mesh filename=sr_description/hand/model/knuckle.dae scale=0.001 0.001 0.001
- link ffmiddle: geometry collision box size=0.008 0.008 0.015; visual mesh filename=sr_description/hand/model/F2.dae scale=0.001 0.001 0.001
- link ffproximal: geometry collision box size=0.008 0.008 0.04; visual mesh filename=sr_description/hand/model/F3.dae scale=0.001 0.001 0.001
- link forearm: geometry collision cylinder length=0.180 radius=0.06; visual mesh filename=sr_description/hand/model/forearm.dae scale=0.001 0.001 0.001
- link lfdistal: geometry collision mesh filename=sr_description/hand/model/F1.dae scale=0.001 0.001 0.001; visual mesh filename=sr_description/hand/model/F1.dae scale=0.001 0.001 0.001
- link lfknuckle: geometry collision box size=0.005 0.005 0.005; visual mesh filename=sr_description/hand/model/knuckle.dae scale=0.001 0.001 0.001
- link lfmetacarpal: geometry collision box size=0.008 0.008 0.03; visual mesh filename=sr_description/hand/model/lfmetacarpal.dae scale=0.001 0.001 0.001
- link lfmiddle: geometry collision box size=0.008 0.008 0.015; visual mesh filename=sr_description/hand/model/F2.dae scale=0.001 0.001 0.001
- link lfproximal: geometry collision box size=0.008 0.008 0.04; visual mesh filename=sr_description/hand/model/F3.dae scale=0.001 0.001 0.001
- link mfdistal: geometry collision mesh filename=sr_description/hand/model/F1.dae scale=0.001 0.001 0.001; visual mesh filename=sr_description/hand/model/F1.dae scale=0.001 0.001 0.001
- link mfknuckle: geometry collision box size=0.005 0.005 0.005; visual mesh filename=sr_description/hand/model/knuckle.dae scale=0.001 0.001 0.001
- link mfmiddle: geometry collision box size=0.008 0.008 0.015; visual mesh filename=sr_description/hand/model/F2.dae scale=0.001 0.001 0.001
- link mfproximal: geometry collision box size=0.008 0.008 0.04; visual mesh filename=sr_description/hand/model/F3.dae scale=0.001 0.001 0.001
- link palm: geometry collision box size=0.05 0.02 0.07; visual mesh filename=sr_description/hand/model/palm.dae scale=0.001 0.001 0.001
- link rfdistal: geometry collision mesh filename=sr_description/hand/model/F1.dae scale=0.001 0.001 0.001; visual mesh filename=sr_description/hand/model/F1.dae scale=0.001 0.001 0.001
- link rfknuckle: geometry collision box size=0.005 0.005 0.005; visual mesh filename=sr_description/hand/model/knuckle.dae scale=0.001 0.001 0.001
- link rfmiddle: geometry collision box size=0.008 0.008 0.015; visual mesh filename=sr_description/hand/model/F2.dae scale=0.001 0.001 0.001
- link rfproximal: geometry collision box size=0.008 0.008 0.04; visual mesh filename=sr_description/hand/model/F3.dae scale=0.001 0.001 0.001
- link shadowarm_base: geometry collision mesh filename=sr_description/arm/model/arm_base.dae scale=0.001 0.001 0.001; visual mesh filename=sr_description/arm/model/arm_base.dae scale=0.001 0.001 0.001
- link shadowarm_handsupport: geometry collision cylinder length=0.001 radius=0.06; visual mesh filename=sr_description/arm/model/elbow_rotate_motor.dae scale=0.001 0.001 0.001
- link shadowarm_lowerarm: geometry collision mesh filename=sr_description/arm/model/elbow_flex.dae scale=0.001 0.001 0.001; visual mesh filename=sr_description/arm/model/elbow_flex.dae scale=0.001 0.001 0.001
- link shadowarm_trunk: geometry collision mesh filename=sr_description/arm/model/arm_trunk.dae scale=0.001 0.001 0.001; visual mesh filename=sr_description/arm/model/arm_trunk.dae scale=0.001 0.001 0.001
- link shadowarm_upperarm: geometry collision mesh filename=sr_description/arm/model/upper_arm.dae scale=0.001 0.001 0.001; visual mesh filename=sr_description/arm/model/upper_arm.dae scale=0.001 0.001 0.001
- link thdistal: geometry collision mesh filename=sr_description/hand/model/TH1_z.dae scale=0.001 0.001 0.001; visual mesh filename=sr_description/hand/model/TH1_z.dae scale=0.001 0.001 0.001
- link thmiddle: geometry collision box size=0.008 0.008 0.015; visual mesh filename=sr_description/hand/model/TH2_z.dae scale=0.001 0.001 0.001
- link thproximal: geometry collision box size=0.008 0.008 0.020; visual mesh filename=sr_description/hand/model/TH3_z.dae scale=0.001 0.001 0.001
- link wrist: geometry collision box size=0.02 0.02 0.02; visual mesh filename=sr_description/hand/model/wrist.dae scale=0.001 0.001 0.001

File: data/urdf/shadow_hand_john/model_forearm_and_hand.urdf (robot description, URDF)
Before this commit: robot arm_and_hand, 33 links, 32 joints
Links:
- link ffdistal: geometry collision mesh filename=sr_description/hand/model/F1.dae scale=0.001 0.001 0.001; visual mesh filename=sr_description/hand/model/F1.dae scale=0.001 0.001 0.001
- link ffknuckle: geometry collision box size=0.005 0.005 0.005; visual mesh filename=sr_description/hand/model/knuckle.dae scale=0.001 0.001 0.001
- link ffmiddle: geometry collision box size=0.008 0.008 0.015; visual mesh filename=sr_description/hand/model/F2.dae scale=0.001 0.001 0.001
- link ffproximal: geometry collision box size=0.008 0.008 0.04; visual mesh filename=sr_description/hand/model/F3.dae scale=0.001 0.001 0.001
- link forearm: geometry collision cylinder length=0.180 radius=0.06; visual mesh filename=sr_description/hand/model/forearm.dae scale=0.001 0.001 0.001
- link lfdistal: geometry collision mesh filename=sr_description/hand/model/F1.dae scale=0.001 0.001 0.001; visual mesh filename=sr_description/hand/model/F1.dae scale=0.001 0.001 0.001
- link lfknuckle: geometry collision box size=0.005 0.005 0.005; visual mesh filename=sr_description/hand/model/knuckle.dae scale=0.001 0.001 0.001
- link lfmetacarpal: geometry collision box size=0.008 0.008 0.03; visual mesh filename=sr_description/hand/model/lfmetacarpal.dae scale=0.001 0.001 0.001
- link lfmiddle: geometry collision box size=0.008 0.008 0.015; visual mesh filename=sr_description/hand/model/F2.dae scale=0.001 0.001 0.001
- link lfproximal: geometry collision box size=0.008 0.008 0.04; visual mesh filename=sr_description/hand/model/F3.dae scale=0.001 0.001 0.001
- link mfdistal: geometry collision mesh filename=sr_description/hand/model/F1.dae scale=0.001 0.001 0.001; visual mesh filename=sr_description/hand/model/F1.dae scale=0.001 0.001 0.001
- link mfknuckle: geometry collision box size=0.005 0.005 0.005; visual mesh filename=sr_description/hand/model/knuckle.dae scale=0.001 0.001 0.001
- link mfmiddle: geometry collision box size=0.008 0.008 0.015; visual mesh filename=sr_description/hand/model/F2.dae scale=0.001 0.001 0.001
- link mfproximal: geometry collision box size=0.008 0.008 0.04; visual mesh filename=sr_description/hand/model/F3.dae scale=0.001 0.001 0.001
- link palm: geometry collision box size=0.05 0.02 0.07; visual mesh filename=sr_description/hand/model/palm.dae scale=0.001 0.001 0.001
- link rfdistal: geometry collision mesh filename=sr_description/hand/model/F1.dae scale=0.001 0.001 0.001; visual mesh filename=sr_description/hand/model/F1.dae scale=0.001 0.001 0.001
- link rfknuckle: geometry collision box size=0.005 0.005 0.005; visual mesh filename=sr_description/hand/model/knuckle.dae scale=0.001 0.001 0.001
- link rfmiddle: geometry collision box size=0.008 0.008 0.015; visual mesh filename=sr_description/hand/model/F2.dae scale=0.001 0.001 0.001
- link rfproximal: geometry collision box size=0.008 0.008 0.04; visual mesh filename=sr_description/hand/model/F3.dae scale=0.001 0.001 0.001
- link shadowarm_handsupport: geometry collision cylinder length=0.001 radius=0.06; visual mesh filename=sr_description/arm/model/elbow_rotate_motor.dae scale=0.001 0.001 0.001
- link shadowarm_lowerarm: geometry collision mesh filename=sr_description/arm/model/elbow_flex.dae scale=0.001 0.001 0.001; visual mesh filename=sr_description/arm/model/elbow_flex.dae scale=0.001 0.001 0.001
- link thdistal: geometry collision mesh filename=sr_description/hand/model/TH1_z.dae scale=0.001 0.001 0.001; visual mesh filename=sr_description/hand/model/TH1_z.dae scale=0.001 0.001 0.001
- link thmiddle: geometry collision box size=0.008 0.008 0.015; visual mesh filename=sr_description/hand/model/TH2_z.dae scale=0.001 0.001 0.001
- link thproximal: geometry collision box size=0.008 0.008 0.020; visual mesh filename=sr_description/hand/model/TH3_z.dae scale=0.001 0.001 0.001
- link wrist: geometry collision box size=0.02 0.02 0.02; visual mesh filename=sr_description/hand/model/wrist.dae scale=0.001 0.001 0.001

File: data/urdf/shadow_hand_john/model_forearm_and_hand_JS.urdf (robot description, URDF)
Before this commit: robot arm_and_hand, 32 links, 32 joints
Links:
- added link shadowarm_lowerarm, mass 0.5; collision mesh filename=sr_description/arm/model/elbow_flex.dae scale=0.001 0.001 0.001; visual mesh filename=sr_description/arm/model/elbow_flex.dae scale=0.001 0.001 0.001
- link ffdistal: geometry collision mesh filename=sr_description/hand/model/F1.dae scale=0.001 0.001 0.001; visual mesh filename=sr_description/hand/model/F1.dae scale=0.001 0.001 0.001
- link ffknuckle: geometry collision box size=0.005 0.005 0.005; visual mesh filename=sr_description/hand/model/knuckle.dae scale=0.001 0.001 0.001
- link ffmiddle: geometry collision box size=0.008 0.008 0.015; visual mesh filename=sr_description/hand/model/F2.dae scale=0.001 0.001 0.001
- link ffproximal: geometry collision box size=0.008 0.008 0.04; visual mesh filename=sr_description/hand/model/F3.dae scale=0.001 0.001 0.001
- link forearm: geometry collision cylinder length=0.180 radius=0.06; visual mesh filename=sr_description/hand/model/forearm.dae scale=0.001 0.001 0.001
- link lfdistal: geometry collision mesh filename=sr_description/hand/model/F1.dae scale=0.001 0.001 0.001; visual mesh filename=sr_description/hand/model/F1.dae scale=0.001 0.001 0.001
- link lfknuckle: geometry collision box size=0.005 0.005 0.005; visual mesh filename=sr_description/hand/model/knuckle.dae scale=0.001 0.001 0.001
- link lfmetacarpal: geometry collision box size=0.008 0.008 0.03; visual mesh filename=sr_description/hand/model/lfmetacarpal.dae scale=0.001 0.001 0.001
- link lfmiddle: geometry collision box size=0.008 0.008 0.015; visual mesh filename=sr_description/hand/model/F2.dae scale=0.001 0.001 0.001
- link lfproximal: geometry collision box size=0.008 0.008 0.04; visual mesh filename=sr_description/hand/model/F3.dae scale=0.001 0.001 0.001
- link mfdistal: geometry collision mesh filename=sr_description/hand/model/F1.dae scale=0.001 0.001 0.001; visual mesh filename=sr_description/hand/model/F1.dae scale=0.001 0.001 0.001
- link mfknuckle: geometry collision box size=0.005 0.005 0.005; visual mesh filename=sr_description/hand/model/knuckle.dae scale=0.001 0.001 0.001
- link mfmiddle: geometry collision box size=0.008 0.008 0.015; visual mesh filename=sr_description/hand/model/F2.dae scale=0.001 0.001 0.001
- link mfproximal: geometry collision box size=0.008 0.008 0.04; visual mesh filename=sr_description/hand/model/F3.dae scale=0.001 0.001 0.001
- link palm: geometry collision box size=0.05 0.02 0.07; visual mesh filename=sr_description/hand/model/palm.dae scale=0.001 0.001 0.001
- link rfdistal: geometry collision mesh filename=sr_description/hand/model/F1.dae scale=0.001 0.001 0.001; visual mesh filename=sr_description/hand/model/F1.dae scale=0.001 0.001 0.001
- link rfknuckle: geometry collision box size=0.005 0.005 0.005; visual mesh filename=sr_description/hand/model/knuckle.dae scale=0.001 0.001 0.001
- link rfmiddle: geometry collision box size=0.008 0.008 0.015; visual mesh filename=sr_description/hand/model/F2.dae scale=0.001 0.001 0.001
- link rfproximal: geometry collision box size=0.008 0.008 0.04; visual mesh filename=sr_description/hand/model/F3.dae scale=0.001 0.001 0.001
- link shadowarm_handsupport: geometry collision cylinder length=0.001 radius=0.06; visual mesh filename=sr_description/arm/model/elbow_rotate_motor.dae scale=0.001 0.001 0.001
- link thdistal: geometry collision mesh filename=sr_description/hand/model/TH1_z.dae scale=0.001 0.001 0.001; visual mesh filename=sr_description/hand/model/TH1_z.dae scale=0.001 0.001 0.001
- link thmiddle: geometry collision box size=0.008 0.008 0.015; visual mesh filename=sr_description/hand/model/TH2_z.dae scale=0.001 0.001 0.001
- link thproximal: geometry collision box size=0.008 0.008 0.020; visual mesh filename=sr_description/hand/model/TH3_z.dae scale=0.001 0.001 0.001
- link wrist: geometry collision box size=0.02 0.02 0.02; visual mesh filename=sr_description/hand/model/wrist.dae scale=0.001 0.001 0.001
Joints:
- joint ElbowJSwing: axis (none) -> 0 -1 0; child shadowarm_handsupport -> shadowarm_lowerarm; limit (none) -> lower=0.52 upper=2.09439510239 effort=1000.0 velocity=10.0; type fixed -> revolute
- joint arm_link: origin xyz=0.08 0 0.121 rpy=0 0 2.35619449 -> xyz=0 0 0 rpy=0 0 2.35619449
